File: 56 ch sample-and-hold card v1.1.sch (EAGLE design)
At the start: 143 parts, among them IC1 74HCT4051D, IC10 TL074JT, IC11 74HCT4051D, IC12 TL074JT, IC13 TL074JT, IC14 74HCT4051D, IC15 TL074JT, IC16 TL074JT, IC17 74HCT4051D, IC18 TL074JT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

Commit message: Cleanup of old stuff, renaming repo soon
Other:
- note added: "Changelog v1.1: - Added missing connections from channels to back row of connectors"
Changed lines of the file:
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@@
 <text x="132.08" y="88.9" size="1.778" layer="97">2 x gain, changes 2.5V at
 DAC to 5V at CV buffers</text>
+<text x="0" y="132.08" size="3.81" layer="97">Changelog
+v1.1:
+- Added missing connections from channels to back row of connectors</text>
 </plain>
 <instances>
